File: fc_2026.kicad_sch (KiCad schematic)
At the start: 0 parts

Commit message: Adding base schematics
Other:
- added sheet Autopilot Bus Connector (autopilot_bus_connector.kicad_sch)
- added sheet Barometer 1 (barometer_1.kicad_sch)
- added sheet Barometer 2 (barometer_2.kicad_sch)
- added sheet Can Bus Connector (can_bus_connector.kicad_sch)
- added sheet Debug Connector (debug_connector.kicad_sch)
- added sheet Ethernet Connection (ethernet_connection.kicad_sch)
- added sheet FMU MCU (fmu_mcu.kicad_sch)
- added sheet GPS Connectors (gps_connectors.kicad_sch)
- added sheet I2C Expansion Connectors (i2c_expansion.kicad_sch)
- added sheet IMU 1 (imu_1.kicad_sch)
- added sheet IMU 2 (imu_2.kicad_sch)
- added sheet IMU 3 (imu_3.kicad_sch)
- added sheet PWM Output Connectors (pwm_output_connectors.kicad_sch)
- added sheet Power Connector (power_connector.kicad_sch)
- added sheet Power Zone 1 (power_zone_1.kicad_sch)
- added sheet Power Zone 2 (power_zone_2.kicad_sch)
- added sheet Power Zone 3 (power_zone_3.kicad_sch)
- added sheet RC Input Connector (rc_input_connector.kicad_sch)
- added sheet Telemetry 1 (telemetry_1.kicad_sch)
- added sheet Telemetry 2 (telemetry_2.kicad_sch)
